File: Modules/RW_EM_DLF_A/PCB/RW_EM_DLF_A.kicad_pcb (KiCad board)
At the start: 2 copper layers, 60 x 100 mm, 70 parts, among them J1 PJ301M-12, J2 PJ301M-12, J3 IDC_02x05, J4 PJ301M-12, J5 PJ301M-12, J6 PJ301M-12, U1 TL074, U2 TL074

Commit message: Added RW_EM_MIXER_A
Other:
- board text added: "REV 2022-10-19"
- board text removed: "REV 2022-10-18"
Changed lines of the file:
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@@
     (effects (font (size 1 1) (thickness 0.16)) (justify mirror))
   )
-  (gr_text "REV 2022-10-18" (at 178.435 58.42 90) (layer "B.SilkS")
+  (gr_text "REV 2022-10-19" (at 178.435 58.42 90) (layer "B.SilkS")
     (effects (font (size 1 1) (thickness 0.16)) (justify mirror))
   )
