File: Modules/RW_EM_SH_NOISE_A/PCB/RW_EM_SH_NOISE_A.kicad_sch (KiCad schematic)
At the start: 68 parts, among them J1 IDC_02x05, J2 PJ301M-12, J3 PJ301M-12, J4 PJ301M-12, J5 PJ301M-12, J6 PJ301M-12, J7 PJ301M-12, Q1 BC548, Q2 BC548, Q3 J113, U1 TL074, U2 TL072

Commit message: Added helpful information to the main readme. Also added pictures to some modules
Parts:
- R26: value 22k -> 20k
Changed lines of the file:
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@@
       (effects (font (size 1.27 1.27)) (justify left))
     )
-    (property "Value" "22k" (id 1) (at 166.37 102.87 0)
+    (property "Value" "20k" (id 1) (at 166.37 102.87 0)
       (effects (font (size 1.27 1.27)) (justify left))
     )
@@
     )
     (path "/4b65360f-488b-438c-960a-e2e6bae5019c"
-      (reference "R26") (unit 1) (value "22k") (footprint "Resistor_THT:R_Axial_DIN0207_L6.3mm_D2.5mm_P2.54mm_Vertical")
+      (reference "R26") (unit 1) (value "20k") (footprint "Resistor_THT:R_Axial_DIN0207_L6.3mm_D2.5mm_P2.54mm_Vertical")
     )
     (path "/3e3e99ee-bb1e-406a-8e4d-b7328208b1fb"
