File: Modules/RW_EM_SH_NOISE_A/PCB/RW_EM_SH_NOISE_A.kicad_pcb (KiCad board)
At the start: 2 copper layers, 50 x 100 mm, 68 parts, among them J1 IDC_02x05, J2 PJ301M-12, J3 PJ301M-12, J4 PJ301M-12, J5 PJ301M-12, J6 PJ301M-12, J7 PJ301M-12, Q1 BC548, Q2 BC548, Q3 J113, U1 TL074, U2 TL072

Commit message: Added helpful information to the main readme. Also added pictures to some modules
Parts:
- R26: value 22k -> 20k
