File: Modules/RW_EM_LFO_A/PCB/RW_EM_LFO_A.kicad_pcb (KiCad board)
At the start: 2 copper layers, 20 x 100 mm, 20 parts, among them J1 IDC_02x05, J2 PJ301M-12, SW1 SW_SPDT, U1 TL072

Commit message: Updated all schematics with link to repo. Also updated all readme files
Other:
- board text added: "REV 2022-10-22"
- board text removed: "REV 2022-10-19"
Changed lines of the file:
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@@
     (effects (font (size 0.7 0.7) (thickness 0.12)) (justify mirror))
   )
-  (gr_text "REV 2022-10-19" (at 129.54 106.68 90) (layer "B.SilkS")
+  (gr_text "REV 2022-10-22" (at 129.54 106.68 90) (layer "B.SilkS")
     (effects (font (size 1 1) (thickness 0.16)) (justify mirror))
   )

Commit message: Added RW_EM_DWF_A and RE_EM_WS_A
Other:
- board text added: "https://github.com/ sunfl0w/RW_EM"
- board text removed: "https://github.com/sunfl0w/RW_EM"
Changed lines of the file:
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@@
     (rev "2022-10-19")
     (comment 1 "Licensed under CERN-OHL-S v2+")
+    (comment 2 "https://github.com/sunfl0w/RW_EM")
   )
   (layers
@@
     (property "Sheetname" "")
     (attr through_hole)
-    (fp_text reference "C4" (at 5.08 2.54 90) (layer "B.SilkS")
+    (fp_text reference "C4" (at -2.54 -0.635 90) (layer "B.SilkS")
       (effects (font (size 1 1) (thickness 0.15)) (justify mirror))
     )
@@
     (property "Sheetname" "")
     (attr through_hole)
-    (fp_text reference "C2" (at 5.08 1.27 90) (layer "B.SilkS")
+    (fp_text reference "C2" (at 5.08 0 90) (layer "B.SilkS")
       (effects (font (size 1 1) (thickness 0.15)) (justify mirror))
     )
@@
     (effects (font (size 1 1) (thickness 0.16)) (justify mirror))
   )
-  (gr_text "https://github.com/sunfl0w/RW_EM" (at 146.685 140.97 90) (layer "B.SilkS")
-    (effects (font (size 0.7 0.7) (thickness 0.12)) (justify mirror))
-  )
-  (gr_text "Licensed under CERN-OHL-S v2+" (at 144.145 140.97 90) (layer "B.SilkS")
-    (effects (font (size 0.7 0.7) (thickness 0.12)) (justify mirror))
+  (gr_text "https://github.com/\nsunfl0w/RW_EM" (at 145.415 141.605 90) (layer "B.SilkS")
+    (effects (font (size 1 1) (thickness 0.16)) (justify mirror))
+  )
+  (gr_text "Licensed\nunder\nCERN-OHL-S v2+" (at 137.16 101.6 90) (layer "B.SilkS")
+    (effects (font (size 1 1) (thickness 0.16)) (justify mirror))
   )
   (gr_text "REV 2022-10-22" (at 129.54 106.68 90) (layer "B.SilkS")
