File: Modules/RW_EM_VCAx2_A/PCB/RW_EM_VCAx2_A.kicad_pcb (KiCad board)
At the start: 2 copper layers, 50 x 100 mm, 68 parts, among them J1 IDC_02x05, J2 PJ301M-12, J3 PJ301M-12, J4 PJ301M-12, J5 PJ301M-12, J6 PJ301M-12, J7 PJ301M-12, Q1 BC548, Q2 BC548, Q3 BC548, Q4 BC548, Q5 BC548, Q6 BC548, U1 TL074

Commit message: Added notice for matched resistors. Added small silkscreen changes to VCO_A and VCAx2_A
Other:
- board text added: "RV3 and RV4 TRANSISTOR TRIM"
- board text added: "RV5 and RV6 0V TRIM"
Changed lines of the file:
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@@
+    (effects (font (size 1 1) (thickness 0.16)) (justify mirror))
+  )
+  (gr_text "RV5 and RV6\n0V TRIM" (at 165.1 133.985) (layer "B.SilkS")
     (effects (font (size 1 1) (thickness 0.16)) (justify mirror))
   )
@@
     (effects (font (size 1 1) (thickness 0.16)) (justify mirror))
   )
-  (gr_text "based on mki x es VCA" (at 157.48 133.985) (layer "B.SilkS")
+  (gr_text "based on mki x es VCA" (at 165.1 127) (layer "B.SilkS")
     (effects (font (size 1 1) (thickness 0.16)) (justify mirror))
   )
@@
     (effects (font (size 1 1) (thickness 0.16)) (justify mirror))
   )
+  (gr_text "RV3 and RV4\nTRANSISTOR TRIM" (at 153.035 133.985) (layer "B.SilkS")
+    (effects (font (size 1 1) (thickness 0.16)) (justify mirror))
+  )
