File: Modules/RW_EM_VCO_A/PCB/RW_EM_VCO_A.kicad_pcb (KiCad board)
At the start: 2 copper layers, 50 x 100 mm, 55 parts, among them J1 PJ301M-12, J2 PJ301M-12, J3 IDC_02x05, J4 PJ301M-12, J5 PJ301M-12, J6 PJ301M-12, Q1 BC558, Q2 BC548, U1 TL074, U2 40106

Commit message: Added notice for matched resistors. Added small silkscreen changes to VCO_A and VCAx2_A
Other:
- board text added: "TUNE TRIMMER"
Changed lines of the file:
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@@
+    (effects (font (size 1 1) (thickness 0.16)) (justify mirror))
+  )
+  (gr_text "TUNE\nTRIMMER" (at 114.3 123.19) (layer "B.SilkS")
     (effects (font (size 1 1) (thickness 0.16)) (justify mirror))
   )
